Commit message: task 179: added new launch files for accel tracks, requires EUFS sim in catkin ws

File: urdf/tortoisebot.urdf.xacro (robot description, xacro)
@@ -123,6 +123,6 @@
     <!-- Mount Ouster OS1-64 LiDAR -->
     <xacro:include filename="$(find ouster_description)/urdf/OS1-64.urdf.xacro" />
-    <OS1-64 parent="base_link" name="os1_sensor" hz="10" samples="220">
-        <origin xyz="0 0 1.2" rpy="0 0 0" />
+    <OS1-64 parent="base_link" name="os1_sensor" hz="10" samples="512">
+        <origin xyz="0 0 0.3" rpy="0 0 0" />
     </OS1-64>
     <!-- Load differential drive plugin -->
